Commit message: Adding base plate and correct scaling of the wheels
Signed-off-by: Kevin Trejos Vargas <trejkev@gmail.com>

File: urdf/mecanum_wheel.xacro (robot description, xacro)
@@ -26,10 +26,10 @@
                 <xacro:if value="${reflect}">
                     <geometry>
-                        <mesh filename="package://cerlab_mecanum/meshes/wheels/omni_wheel_1.dae" />
+                        <mesh filename="package://cerlab_mecanum/meshes/omni_wheel_1.dae" scale="0.8 0.8 0.8"/>
                     </geometry>
                 </xacro:if>
                 <xacro:unless value="${reflect}">
                     <geometry>
-                        <mesh filename="package://cerlab_mecanum/meshes/wheels/omni_wheel_2.dae" />
+                        <mesh filename="package://cerlab_mecanum/meshes/omni_wheel_2.dae" scale="0.8 0.8 0.8"/>
                     </geometry>
                 </xacro:unless>

File: urdf/robot.xacro (robot description, xacro)
@@ -16,5 +16,5 @@
     <xacro:include filename="$(find cerlab_mecanum)/urdf/robot.gazebo"/>
     <link name="base_footprint"></link>
-    <!-- Main body -->
+    <!-- Adding the main body -->
     <joint name="base_link_joint" type="fixed">
         <origin xyz="0 0 ${wheel_radius + base_link_height/2}" rpy="0 0 0" />
@@ -26,5 +26,4 @@
             <origin rpy=" 0 0 0" xyz="0 0 0"/>
             <geometry>
-                <!-- <box size="${base_link_length} ${base_link_width} ${base_link_height}"/> -->
                 <mesh filename="package://cerlab_mecanum/meshes/escarabajo_armado.stl" scale="0.001 0.001 0.001"/>
             </geometry>
@@ -47,213 +46,48 @@
         </inertial>
     </link>
-    <!-- Wheel PP -->
-    <joint name="joint_wheel_xpyp_shaft" type="fixed">
-        <parent link="base_link"/>
-        <child link="wheel_xpyp_shaft"/>]
-        <origin xyz="${base_link_length/2} ${base_link_width/2-0.065} ${-base_link_height/2}" rpy="0 ${PI/2} 0"/>
+    <!-- Adding the base of the main body (visual purposes only) -->
+    <joint name="base_plate_link_joint" type="fixed">
+        <origin xyz="0 0.03 ${wheel_radius + 0.02}" rpy="0 0 0" />
+        <parent link="base_footprint"/>
+        <child link="base_plate_link" />
     </joint>
-    <link name="wheel_xpyp_shaft">
+    <link name="base_plate_link">
         <visual>
-            <origin xyz="0 0 0" rpy="0 0 0"/>
+            <origin rpy=" 0 0 0" xyz="0 0 0"/>
             <geometry>
-                <cylinder radius="${shaft_radius}" length="${shaft_length}"/>
+                <box size="${base_link_length} ${base_link_width - 0.05} 0.001" />
             </geometry>
-            <material name="black"/>
+            <material name="dark_grey"/>
         </visual>
         <collision>
-            <origin xyz="0 0 0 " rpy="0 0 0"/>
+            <origin rpy=" 0 0 0" xyz="0 0 0"/>
             <geometry>
-                <cylinder radius="${shaft_radius}" length="${shaft_length}"/>
-            </geometry>
-        </collision>
-    </link>
-    <xacro:omni_wheel prefix="wheel_xpyp" parent="base_link" reflect="false">
-        <origin xyz="${base_link_length/2 + 0.05} ${base_link_width/2-0.065} ${-base_link_height/2}" rpy="0 ${PI/2} 0"/>
-    </xacro:omni_wheel>
-    <!-- <joint name="wheel_xpyp_joint" type="continuous">
-        <origin xyz="${base_link_length/2 + 0.05} ${base_link_width/2-0.065} ${-base_link_height/2}" rpy="0 ${PI/2} 0"/>
-        <parent link="base_link"/>
-        <child link="wheel_xpyp"/>
-        <axis xyz="0 0 1"/>
-    </joint>
-    <link name="wheel_xpyp">
-        <visual>
-            <origin xyz="0 0 ${wheel_width/2}" rpy="0 0 0"/>
-            <geometry>
-                <mesh filename="package://cerlab_mecanum/meshes/mecanum_wheel.stl" scale="0.001 0.001 0.001"/>
-            </geometry>
-            <material name="black"/>
-        </visual>
-        <collision>
-            <origin xyz="0 0 ${wheel_width/2}" rpy="0 0 0"/>
-            <geometry>
-                <cylinder radius="${wheel_radius}" length="${wheel_width}"/>
+                <mesh filename="package://cerlab_mecanum/meshes/escarabajo_armado.stl" scale="0.001 0.001 0.001"/>
             </geometry>
         </collision>
         <inertial>
-            <origin xyz="0 0 ${wheel_width/2}"/>
-            <mass value="1"/>
-            <inertia ixx="100" ixy="0.0" ixz="0.0"
-                     iyy="100" iyz="0.0"
-                     izz="100"/>
-        </inertial>
-    </link> -->
-    <!-- Wheel NP -->
-    <joint name="joint_wheel_xnyp_shaft" type="fixed">
-        <parent link="base_link"/>
-        <child link="wheel_xnyp_shaft"/>
-        <origin xyz="${-base_link_length/2} ${base_link_width/2-0.065} ${-base_link_height/2}" rpy="0 ${-PI/2} 0"/>
-    </joint>
-    <link name="wheel_xnyp_shaft">
-        <visual>
             <origin xyz="0 0 0" rpy="0 0 0"/>
-            <geometry>
-                <cylinder radius="${shaft_radius}" length="${shaft_length}"/>
-            </geometry>
-            <material name="black"/>
-        </visual>
-        <collision>
-            <origin xyz="0 0 0 " rpy="0 0 0"/>
-            <geometry>
-                <cylinder radius="${shaft_radius}" length="${shaft_length}"/>
-            </geometry>
-        </collision>
-    </link>
-    <joint name="wheel_xnyp_joint" type="continuous">
-        <origin xyz="${-base_link_length/2 - 0.05} ${base_link_width/2-0.065} ${-base_link_height/2}" rpy="0 ${-PI/2} 0"/>
-        <parent link="base_link"/>
-        <child link="wheel_xnyp" />
-        <axis xyz="0 0 1"/>
-    </joint>
-    <link name="wheel_xnyp">
-        <visual>
-            <origin xyz="0 0 ${wheel_width/2}" rpy="0 0 0" />
-            <geometry>
-                <mesh filename="package://cerlab_mecanum/meshes/mecanum_wheel.stl" scale="0.001 0.001 0.001"/>
-            </geometry>
-            <material name="black" />
-        </visual>
-        <collision>
-            <origin xyz="0 0 ${wheel_width/2}" rpy="0 0 0"/>
-            <geometry>
-                <cylinder radius="${wheel_radius}" length="${wheel_width}"/>
-            </geometry>
-        </collision>
-        <inertial>
-            <origin xyz="0 0 ${wheel_width/2}" rpy="0 0 0"/>
-            <mass value="1.6"/>
-            <!-- Inertia based on cylinder -->
+            <mass value="8.0"/>
             <inertia
-                ixx="0.000324824" ixy="0" ixz="0"
-                iyy="0.000480000" iyz="0"
-                izz="0.000324824"
+                ixx="0.1" ixy="0" ixz="0"
+                iyy="0.1" iyz="0"
+                izz="0.1"
             />
         </inertial>
     </link>
-    <!-- Wheel PN -->
-    <joint name="joint_wheel_xpyn_shaft" type="fixed">
-        <parent link="base_link"/>
-        <child link="wheel_xpyn_shaft"/>
-        <origin xyz="${base_link_length/2} ${-base_link_width/2+0.095} ${-base_link_height/2}" rpy="0 ${PI/2} 0"/>
-    </joint>
-    <link name="wheel_xpyn_shaft">
-        <visual>
-            <origin xyz="0 0 0" rpy="0 0 0"/>
-            <geometry>
-                <cylinder radius="${shaft_radius}" length="${shaft_length}"/>
-            </geometry>
-            <material name="black"/>
-        </visual>
-        <collision>
-            <origin xyz="0 0 0 " rpy="0 0 0"/>
-            <geometry>
-                <cylinder radius="${shaft_radius}" length="${shaft_length}"/>
-            </geometry>
-        </collision>
-    </link>
-    <joint name="wheel_xpyn_joint" type="continuous">
-        <origin xyz="${base_link_length/2 + 0.05} ${-base_link_width/2+0.095} ${-base_link_height/2}" rpy="0 ${PI/2} 0"/>
-        <parent link="base_link"/>
-        <child link="wheel_xpyn" />
-        <axis xyz="0 0 1"/>
-    </joint>
-    <link name="wheel_xpyn">
-        <visual>
-            <origin xyz="0 0 ${wheel_width/2}" rpy="0 0 0" />
-            <geometry>
-                <mesh filename="package://cerlab_mecanum/meshes/mecanum_wheel.stl" scale="0.001 0.001 0.001"/>
-            </geometry>
-            <material name="black" />
-        </visual>
-        <collision>
-            <origin xyz="0 0 ${wheel_width/2}" rpy="0 0 0"/>
-            <geometry>
-                <cylinder radius="${wheel_radius}" length="${wheel_width}"/>
-            </geometry>
-        </collision>
-        <inertial>
-            <origin xyz="0 0 ${wheel_width/2}" rpy="0 0 0"/>
-            <mass value="1.6"/>
-            <!-- Inertia based on cylinder -->
-            <inertia
-                ixx="0.000324824" ixy="0" ixz="0"
-                iyy="0.000480000" iyz="0"
-                izz="0.000324824"
-            />
-        </inertial>
-    </link>
-    <!-- Wheel NN -->
-    <joint name="joint_wheel_xnyn_shaft" type="fixed">
-        <parent link="base_link"/>
-        <child link="wheel_xnyn_shaft"/>
-        <origin xyz="${-base_link_length/2} ${-base_link_width/2+0.095} ${-base_link_height/2}" rpy="0 ${-PI/2} 0"/>
-    </joint>
-    <link name="wheel_xnyn_shaft">
-        <visual>
-            <origin xyz="0 0 0" rpy="0 0 0"/>
-            <geometry>
-                <cylinder radius="${shaft_radius}" length="${shaft_length}"/>
-            </geometry>
-            <material name="black"/>
-        </visual>
-        <collision>
-            <origin xyz="0 0 0 " rpy="0 0 0"/>
-            <geometry>
-                <cylinder radius="${shaft_radius}" length="${shaft_length}"/>
-            </geometry>
-        </collision>
-    </link>
-    <joint name="wheel_xnyn_joint" type="fixed">
-        <origin xyz="${-base_link_length/2 - 0.05} ${-base_link_width/2+0.095} ${-base_link_height/2}" rpy="0 ${-PI/2} 0"/>
-        <parent link="base_link"/>
-        <child link="wheel_xnyn" />
-        <axis xyz="0 0 1"/>
-    </joint>
-    <link name="wheel_xnyn">
-        <visual>
-            <origin xyz="0 0 ${wheel_width/2}" rpy="0 0 0" />
-            <geometry>
-                <mesh filename="package://cerlab_mecanum/meshes/mecanum_wheel.stl" scale="0.001 0.001 0.001"/>
-            </geometry>
-            <material name="black" />
-        </visual>
-        <collision>
-            <origin xyz="0 0 ${wheel_width/2}" rpy="0 0 0"/>
-            <geometry>
-                <cylinder radius="${wheel_radius}" length="${wheel_width}"/>
-            </geometry>
-        </collision>
-        <inertial>
-            <origin xyz="0 0 ${wheel_width/2}" rpy="0 0 0"/>
-            <mass value="1.6"/>
-            <!-- Inertia based on cylinder -->
-            <inertia
-                ixx="0.000324824" ixy="0" ixz="0"
-                iyy="0.000480000" iyz="0"
-                izz="0.000324824"
-            />
-        </inertial>
-    </link>
-    <!-- LiDAR sensors -->
+    <!-- Adding mecanum wheels -->
+    <xacro:omni_wheel prefix="xpyp" parent="base_link" reflect="false">
+        <origin xyz="${base_link_length/2 + wheel_width/2 + 0.01} ${base_link_width/2-0.065} ${-base_link_height/2 + 0.02}" rpy="0 0 ${PI/2}"/>
+    </xacro:omni_wheel>
+    <xacro:omni_wheel prefix="xnyp" parent="base_link" reflect="true">
+        <origin xyz="${-base_link_length/2 - wheel_width/2 - 0.01} ${base_link_width/2-0.065} ${-base_link_height/2 + 0.02}" rpy="0 0 ${PI/2}"/>
+    </xacro:omni_wheel>
+    <xacro:omni_wheel prefix="xpyn" parent="base_link" reflect="true">
+        <origin xyz="${base_link_length/2 + wheel_width/2 + 0.01} ${-base_link_width/2+0.095} ${-base_link_height/2 + 0.02}" rpy="0 0 ${PI/2}"/>
+    </xacro:omni_wheel>
+    <xacro:omni_wheel prefix="xnyn" parent="base_link" reflect="false">
+        <origin xyz="${-base_link_length/2 - wheel_width/2 - 0.01} ${-base_link_width/2+0.095} ${-base_link_height/2 + 0.02}" rpy="0 0 ${PI/2}"/>
+    </xacro:omni_wheel>
+    <!-- Adding LiDAR sensors -->
     <joint name="front_scan_joint" type="fixed">
         <parent link="base_link"/>
@@ -286,5 +120,4 @@
         <parent link="base_link"/>
         <child link="base_scan_back"/>
-        <!-- <origin xyz="0.09 ${-base_link_width/2+0.115} ${base_link_height/2+0.1}" rpy="0 0 0"/> -->
         <origin xyz="0 ${-base_link_width/2+0.1} ${base_link_height/2+0.05}" rpy="0 0 0"/>
     </joint>
