Commit message: Removing unnecessary variablesf
This change is removing some of the unnecessary tags in the code.

Signed-off-by: Kevin Trejos Vargas <trejkev@gmail.com>

File: urdf/robot.xacro (robot description, xacro)
@@ -12,20 +12,4 @@
     <xacro:property name="shaft_length" value="0.1"       />
     <xacro:property name="shaft_radius" value="0.005"     />
-    <!-- LiDAR sensor parameters -->
-    <xacro:property name="s1_x_axis_front_location" value="0"  />
-    <xacro:property name="s1_y_axis_front_location" value="20" />
-    <xacro:property name="s2_x_axis_front_location" value="0"  />
-    <xacro:property name="s2_y_axis_front_location" value="-20"/>
-    <!-- Joint limits parameters -->
-    <!-- Main wheel limits -->
-    <xacro:property name="main_wheel_max_rev"      value="3.14" />
-    <xacro:property name="main_wheel_min_rev"      value="-3.14"/>
-    <xacro:property name="main_wheel_max_velocity" value="3.14" />
-    <xacro:property name="main_wheel_max_effort"   value="300"  />
-    <!-- Rollers limits-->
-    <xacro:property name="rollers_max_rev"      value="3.14" />
-    <xacro:property name="rollers_min_rev"      value="-3.14"/>
-    <xacro:property name="rollers_max_velocity" value="3.14" />
-    <xacro:property name="rollers_max_effort"   value="300"  />
     <xacro:include filename="$(find cerlab_mecanum)/urdf/robot.gazebo"/>
     <link name="base_footprint"></link>
@@ -62,5 +46,4 @@
     </link>
     <!-- Wheel PP -->
-    <!-- The shaft is just for visual effect -->
     <joint name="joint_wheel_xpyp_shaft" type="fixed">
         <parent link="base_link"/>
@@ -272,5 +255,4 @@
         <parent link="base_link"/>
         <child link="base_scan_front"/>
-        <!-- <origin xyz="0.09 ${base_link_width/2-0.004} ${base_link_height/2+0.1}" rpy="0 0 0"/> era 0.04 en z y 0 en x -->
         <origin xyz="0 ${base_link_width/2-0.046} ${base_link_height/2+0.05}" rpy="0 0 0"/>
     </joint>

Commit message: Adding mecanum wheel model

File: urdf/robot.xacro (robot description, xacro)
@@ -1,4 +1,6 @@
 <?xml version="1.0"?>
 <robot xmlns:xacro="http://www.ros.org/wiki/xacro" name="cerlab_mecanum">
+    <!-- Bring mecanum wheel to the model -->
+    <xacro:include filename="$(find cerlab_mecanum)/urdf/mecanum_wheel.xacro" />
     <!-- Robot geometry parameters -->
     <xacro:property name="PI" value="3.1415926535897931" />
@@ -66,5 +68,8 @@
         </collision>
     </link>
-    <joint name="wheel_xpyp_joint" type="continuous">
+    <xacro:omni_wheel prefix="wheel_xpyp" parent="base_link" reflect="false">
+        <origin xyz="${base_link_length/2 + 0.05} ${base_link_width/2-0.065} ${-base_link_height/2}" rpy="0 ${PI/2} 0"/>
+    </xacro:omni_wheel>
+    <!-- <joint name="wheel_xpyp_joint" type="continuous">
         <origin xyz="${base_link_length/2 + 0.05} ${base_link_width/2-0.065} ${-base_link_height/2}" rpy="0 ${PI/2} 0"/>
         <parent link="base_link"/>
@@ -89,10 +94,9 @@
             <origin xyz="0 0 ${wheel_width/2}"/>
             <mass value="1"/>
-            <!-- Inertia based on cylinder -->
             <inertia ixx="100" ixy="0.0" ixz="0.0"
                      iyy="100" iyz="0.0"
                      izz="100"/>
         </inertial>
-    </link>
+    </link> -->
     <!-- Wheel NP -->
     <joint name="joint_wheel_xnyp_shaft" type="fixed">

Commit message: Splitted the descriptors into modules with macros

File: urdf/robot.xacro (robot description, xacro)
@@ -1,6 +1,8 @@
 <?xml version="1.0"?>
 <robot xmlns:xacro="http://www.ros.org/wiki/xacro" name="cerlab_mecanum">
-    <!-- Bring mecanum wheel to the model -->
-    <xacro:include filename="$(find cerlab_mecanum)/urdf/mecanum_wheel.xacro" />
+    <!-- Bring robot parts to the model -->
+    <xacro:include filename="$(find cerlab_mecanum)/urdf/robot_parts/mecanum_wheel.xacro"/>
+    <xacro:include filename="$(find cerlab_mecanum)/urdf/robot_parts/base_link.xacro"    />
+    <xacro:include filename="$(find cerlab_mecanum)/urdf/robot_parts/sensor.xacro"       />
     <!-- Robot geometry parameters -->
     <xacro:property name="PI" value="3.1415926535897931" />
@@ -12,68 +14,13 @@
     <xacro:property name="wheel_radius" value="${0.203/2}"/>
     <xacro:property name="wheel_width"  value="0.078"     />
-    <xacro:property name="shaft_length" value="0.1"       />
-    <xacro:property name="shaft_radius" value="0.005"     />
     <xacro:include filename="$(find cerlab_mecanum)/urdf/robot.gazebo"/>
     <link name="base_footprint"></link>
     <!-- Adding the main body -->
-    <joint name="base_link_joint" type="fixed">
+    <xacro:base_link parent="base_footprint">
         <origin xyz="0 0 ${wheel_radius + base_link_height/2}" rpy="0 0 0" />
-        <parent link="base_footprint"/>
-        <child link="base_link" />
-    </joint>
-    <link name="base_link">
-        <visual>
-            <origin rpy=" 0 0 0" xyz="0 0 0"/>
-            <geometry>
-                <mesh filename="package://cerlab_mecanum/meshes/escarabajo_armado.stl" scale="0.001 0.001 0.001"/>
-            </geometry>
-            <material name="dark_grey"/>
-        </visual>
-        <collision>
-            <origin rpy=" 0 0 0" xyz="0 0 0"/>
-            <geometry>
-                <mesh filename="package://cerlab_mecanum/meshes/escarabajo_armado.stl" scale="0.001 0.001 0.001"/>
-            </geometry>
-        </collision>
-        <inertial>
-            <origin xyz="0 0 0" rpy="0 0 0"/>
-            <mass value="8.0"/>
-            <inertia
-                ixx="0.1" ixy="0" ixz="0"
-                iyy="0.1" iyz="0"
-                izz="0.1"
-            />
-        </inertial>
-    </link>
-    <!-- Adding the base of the main body (visual purposes only) -->
-    <joint name="base_plate_link_joint" type="fixed">
-        <origin xyz="0 0.03 ${wheel_radius + 0.02}" rpy="0 0 0" />
-        <parent link="base_footprint"/>
-        <child link="base_plate_link" />
-    </joint>
-    <link name="base_plate_link">
-        <visual>
-            <origin rpy=" 0 0 0" xyz="0 0 0"/>
-            <geometry>
-                <box size="${base_link_length} ${base_link_width - 0.05} 0.001" />
-            </geometry>
-            <material name="dark_grey"/>
-        </visual>
-        <collision>
-            <origin rpy=" 0 0 0" xyz="0 0 0"/>
-            <geometry>
-                <mesh filename="package://cerlab_mecanum/meshes/escarabajo_armado.stl" scale="0.001 0.001 0.001"/>
-            </geometry>
-        </collision>
-        <inertial>
-            <origin xyz="0 0 0" rpy="0 0 0"/>
-            <mass value="8.0"/>
-            <inertia
-                ixx="0.1" ixy="0" ixz="0"
-                iyy="0.1" iyz="0"
-                izz="0.1"
-            />
-        </inertial>
-    </link>
+    </xacro:base_link>
+    <xacro:base_plate_link parent="base_footprint" length="${base_link_length}" width="${base_link_width - 0.032}" height="0.001">
+        <origin xyz="0 0.023 ${wheel_radius + 0.02}" rpy="0 0 0" />
+    </xacro:base_plate_link>
     <!-- Adding mecanum wheels -->
     <xacro:omni_wheel prefix="xpyp" parent="base_link" reflect="false">
@@ -90,57 +37,9 @@
     </xacro:omni_wheel>
     <!-- Adding LiDAR sensors -->
-    <joint name="front_scan_joint" type="fixed">
-        <parent link="base_link"/>
-        <child link="base_scan_front"/>
+    <xacro:lidar prefix="front" parent="base_link">
         <origin xyz="0 ${base_link_width/2-0.046} ${base_link_height/2+0.05}" rpy="0 0 0"/>
-    </joint>
-    <link name="base_scan_front">
-        <visual>
-            <origin xyz="0 0 0" rpy="0 0 0"/>
-            <geometry>
-                <mesh filename="package://cerlab_mecanum/meshes/hokuyo.stl" scale="1 1 1"/>
-            </geometry>
-            <material name="black"/>
-        </visual>
-        <collision>
-        <origin xyz="0 0 0" rpy="0 0 0"/>
-        <geometry>
-            <cylinder length="0.0315" radius="0.055"/>
-        </geometry>
-        </collision>
-        <inertial>
-        <mass value="0.114" />
-        <origin xyz="0 0 0" />
-        <inertia ixx="0.001" ixy="0.0" ixz="0.0"
-                iyy="0.001" iyz="0.0"
-                izz="0.001" />
-        </inertial>
-    </link>
-    <joint name="back_scan_joint" type="fixed">
-        <parent link="base_link"/>
-        <child link="base_scan_back"/>
+    </xacro:lidar>
+    <xacro:lidar prefix="back" parent="base_link">
         <origin xyz="0 ${-base_link_width/2+0.1} ${base_link_height/2+0.05}" rpy="0 0 0"/>
-    </joint>
-    <link name="base_scan_back">
-        <visual>
-            <origin xyz="0 0 0" rpy="0 0 0"/>
-            <geometry>
-                <mesh filename="package://cerlab_mecanum/meshes/hokuyo.stl" scale="1 1 1"/>
-            </geometry>
-            <material name="black"/>
-        </visual>
-        <collision>
-        <origin xyz="0 0 0" rpy="0 0 0"/>
-        <geometry>
-            <cylinder length="0.0315" radius="0.055"/>
-        </geometry>
-        </collision>
-        <inertial>
-        <mass value="0.114" />
-        <origin xyz="0 0 0" />
-        <inertia ixx="0.001" ixy="0.0" ixz="0.0"
-                iyy="0.001" iyz="0.0"
-                izz="0.001" />
-        </inertial>
-    </link>
+    </xacro:lidar>
 </robot>

Commit message: Added functionality to control the mecanum wheels
Signed-off-by: Kevin Trejos Vargas <trejkev@gmail.com>

File: urdf/robot.xacro (robot description, xacro)
@@ -43,35 +43,3 @@
         <origin xyz="0 ${-base_link_width/2+0.1} ${base_link_height/2+0.05}" rpy="0 0 0"/>
     </xacro:lidar>
-    <!-- Adding the movement control -->
-    <gazebo>
-        <plugin name="movement_controller" filename="libgazebo_ros_planar_move.so">
-            <commandTopic>cmd_vel</commandTopic>
-            <odometryTopic>odom</odometryTopic>
-            <odometryFrame>odom</odometryFrame>
-            <odometryRate>20.0</odometryRate>
-            <robotBaseFrame>base_footprint</robotBaseFrame>
-        </plugin>
-    </gazebo>
-    <!-- <gazebo>
-        <plugin name="gazebo_ros_mecanum_diff_drive" filename="libgazebo_ros_mecanum_drive.so">
-            <commandTopic>cmd_vel</commandTopic>
-            <odometryTopic>odom</odometryTopic>
-            <odometryFrame>odom</odometryFrame>
-            <robotBaseFrame>base_footprint</robotBaseFrame>
-            <LeftRear>xnyn_wheel_joint</LeftRear>
-            <LeftFront>xnyp_wheel_joint</LeftFront>
-            <RightFront>xpyp_wheel_joint</RightFront>
-            <RightRear>xpyn_wheel_joint</RightRear>
-            <odometryRate>20</odometryRate>
-            <publishWheelTF>true</publishWheelTF>
-            <publishWheelJointState>true</publishWheelJointState>
-            <WheelTorque>1</WheelTorque>
-            <WheelSeparationW>0.5</WheelSeparationW>
-            <WheelSeparationL>0.6</WheelSeparationL>
-            <wheelAccel>5</wheelAccel>
-            <wheelDiameter>${wheel_radius*2}</wheelDiameter>
-            <publishOdom>false</publishOdom>
-            <isRollerModel>true</isRollerModel>
-        </plugin>
-    </gazebo> -->
 </robot>

File: urdf/robot_parts/mecanum_wheel.xacro (robot description, xacro)
@@ -19,5 +19,5 @@
             <axis xyz="0 1 0" rpy="0 0 0" />
             <limit effort="100" velocity="100"/>
-            <joint_properties damping="0.0" friction="0.0"/>
+            <dynamics damping="3.0" friction="5.0"/>
         </joint>
         <link name="${prefix}_wheel_link">
@@ -53,15 +53,12 @@
                 <hardwareInterface>hardware_interface/VelocityJointInterface</hardwareInterface>
             </joint>
-            <actuator name="${prefix}_wheel_joint_motor">
-                <mechanicalReduction>1</mechanicalReduction>
-            </actuator>
         </transmission>
         <gazebo reference="${prefix}_wheel_link">
-            <mu1 value="1.0"/>
-            <mu2 value="1.0"/>
-            <kp value="10000000.0" />
-            <kd value="1.0" />
-            <fdir1 value="1 0 0"/>
-            <turnGravityOff>false</turnGravityOff>
+            <gravity>true</gravity>
+            <selfCollide>false</selfCollide>
+            <mu1>30</mu1>
+            <mu2>30</mu2>
+            <kp>1e50</kp>
+            <kd>1e50</kd>
         </gazebo>
     </xacro:macro>

File: urdf/robot_parts/sensor.xacro (robot description, xacro)
@@ -34,5 +34,5 @@
             <sensor type="gpu_ray" name="${prefix}_head_hokuyo_sensor">
                 <pose>0 0 0 0 0 0</pose>
-                <visualize>true</visualize>
+                <visualize>false</visualize>
                 <update_rate>40</update_rate>
                 <ray>
@@ -62,4 +62,10 @@
             </sensor>
         </gazebo>
+        <gazebo reference="${prefix}_lidar_link">
+            <!-- Define friction coefficients and colors -->
+            <mu1>0.2</mu1>
+            <mu2>0.2</mu2>
+            <material>Gazebo/Black</material>
+        </gazebo>
     </xacro:macro>
 </robot>

Commit message: Adding extra visual feedback and correcting 360 degree LiDAR coverage

File: urdf/robot.xacro (robot description, xacro)
@@ -2,8 +2,9 @@
 <robot xmlns:xacro="http://www.ros.org/wiki/xacro" name="cerlab_mecanum">
     <!-- Bring robot parts to the model -->
-    <xacro:include filename="$(find cerlab_mecanum)/urdf/robot_parts/mecanum_wheel.xacro"/>
-    <xacro:include filename="$(find cerlab_mecanum)/urdf/robot_parts/base_link.xacro"    />
-    <xacro:include filename="$(find cerlab_mecanum)/urdf/robot_parts/sensor.xacro"       />
-    <!-- Robot geometry parameters -->
+    <xacro:include filename="$(find cerlab_mecanum)/urdf/robot_parts/mecanum_wheel.xacro"    />
+    <xacro:include filename="$(find cerlab_mecanum)/urdf/robot_parts/base_link.xacro"        />
+    <xacro:include filename="$(find cerlab_mecanum)/urdf/robot_parts/sensor.xacro"           />
+    <xacro:include filename="$(find cerlab_mecanum)/urdf/robot_parts/emergency_button.xacro" />
+    <xacro:include filename="$(find cerlab_mecanum)/urdf/robot_parts/fan.xacro"              />
     <xacro:property name="PI" value="3.1415926535897931" />
     <!-- Robot body ( base link ) parameters -->
@@ -43,3 +44,40 @@
         <origin xyz="0 ${-base_link_width/2+0.1} ${base_link_height/2+0.05}" rpy="0 0 0"/>
     </xacro:lidar>
+    <!-- Adding the emergency buttons (visual feedback only) -->
+    <xacro:emergency_button prefix="front" parent="base_link">
+        <origin xyz="0 ${base_link_width/2+0.017} 0" rpy="${-PI/2} 0 0"/>
+    </xacro:emergency_button>
+    <xacro:emergency_button prefix="back" parent="base_link">
+        <origin xyz="0 ${-base_link_width/2+0.03} 0" rpy="${PI/2} 0 0"/>
+    </xacro:emergency_button>
+    <!-- Adding power button (visual feedback only) -->
+    <joint name="power_button_joint" type="fixed">
+        <parent link="base_link"/>
+        <child link="power_button_link"/>
+        <origin xyz="0 ${-base_link_width/2+0.047} 0.0415" rpy="${PI/2} 0 0"/>
+    </joint>
+        <link name="power_button_link">
+            <visual>
+                <origin rpy=" 0 0 0" xyz="0 0 0"/>
+                <geometry>
+                    <mesh filename="package://cerlab_mecanum/meshes/power_button.stl" scale="0.0011 0.0011 0.0011"/>
+                </geometry>
+            </visual>
+            <collision>
+                <origin rpy=" 0 0 0" xyz="0 0 0"/>
+                <geometry>
+                    <mesh filename="package://cerlab_mecanum/meshes/power_button.stl" scale="0.0011 0.0011 0.0011"/>
+                </geometry>
+            </collision>
+        </link>
+        <gazebo reference="power_button_link">
+            <material>Gazebo/Black</material>
+        </gazebo>
+    <!-- Adding fans (visual feedback only) -->
+    <xacro:fan prefix="left" parent="base_link">
+        <origin xyz="-0.08 ${-base_link_width/2+0.055} ${0.0415/2+0.01}" rpy="${PI/2} 0 0"/>
+    </xacro:fan>
+    <xacro:fan prefix="right" parent="base_link">
+        <origin xyz="0.08 ${-base_link_width/2+0.055} ${0.0415/2+0.01}0" rpy="${PI/2} 0 0"/>
+    </xacro:fan>
 </robot>

File: urdf/robot_parts/sensor.xacro (robot description, xacro)
@@ -1,4 +1,5 @@
 <?xml version="1.0"?>
 <robot name="sensor" xmlns:xacro="http://www.ros.org/wiki/xacro">
+    <xacro:property name="PI" value="3.1415926535897931" />
     <xacro:macro name="lidar" params="prefix parent *origin">
         <joint name="${prefix}_lidar_joint" type="fixed">
@@ -41,6 +42,6 @@
                             <samples>720</samples>
                             <resolution>1</resolution>
-                            <min_angle>-1.570796</min_angle>
-                            <max_angle>1.570796</max_angle>
+                            <min_angle>${-PI}</min_angle>
+                            <max_angle>${PI}</max_angle>
                         </horizontal>
                     </scan>
@@ -63,7 +64,4 @@
         </gazebo>
         <gazebo reference="${prefix}_lidar_link">
-            <!-- Define friction coefficients and colors -->
-            <mu1>0.2</mu1>
-            <mu2>0.2</mu2>
             <material>Gazebo/Black</material>
         </gazebo>
